File: hardware/GridSwitcher_PCB/GridSwitcher_PCB.kicad_pcb (KiCad board)
At the start: 2 copper layers, 160 x 103 mm, 229 parts, among them IC1 INA237AIDGSR, IC2 UCC27536DBVR, IC3 P3T1755DPZ, IC4 P3T1755DPZ, IC5 ESDS304DBVR, IC6 P3T1755DPZ, IC7 P3T1755DPZ, IC8 ESDS304DBVR, IC9 ESDS304DBVR, J1 SSQ-108-03-T-D, J10 Temp Sensor RS485, J11 +24V, J12 SSQ-114-03-T-D, J13 UT_OUT, J14 +3.3V, J15 +5V, J2 SSQ-110-03-T-D, J3 SSQ-108-03-T-D, J4 SSQ-106-03-T-D, J5 Display and Keypad, J6 LEDs, J7 +24V, J8 Battery, J9 SSQ-116-03-T-D, Q1 DMP3013SFV, Q10 DMP3013SFV, Q11 DMP3013SFV, Q12 DMP3013SFV, Q13 DMP3013SFV, Q14 DMP3013SFV, Q15 DMP3013SFV, Q16 DMP3013SFV, Q17 DMP3013SFV, Q2 DMP3013SFV, Q3 DMP3013SFV, Q4 DMP3013SFV, Q5 DMP3013SFV, Q6 DMP3013SFV, Q7 DMP3013SFV, Q8 DMP3013SFV, Q9 DMP3013SFV, U1 74LS09, U10 PC817, U11 PC817, U12 PC817, U13 PC817, U14 PC817, U15 PC817, U16 PC817, U17 PC817, U18 PC817, U19 PC817, U2 74LS09, U20 PC817, U21 PC817, U22 PC817, U23 PC817, U24 PC817, U25 PC817, U26 PC817, U27 PC817, U28 PC817, U29 PC817, U3 PC817, U30 PC817, U31 PC817, U32 PC817, U33 SN65HVD11HD, U34 PC817, U35 PC817, U4 PC817, U5 PC817, U6 PC817, U7 PC817, U8 PC817, U9 PC817

Commit message: -add some changes to schematic, tested the interfaces (uart, spi and i2c) with some test code
Parts:
- added R113: 4.7k, Resistor_SMD:R_0603_1608Metric_Pad0.98x0.95mm_HandSolder, F.Cu at (-2.91, 59.5)
- R107, R11, R16, R21, R26, R31, R36, R41, R46, R51, R56, R6, R61, R66, R71, R76: value 10k -> 100k
- R110, R14, R19, R24, R29, R34, R39, R44, R49, R54, R59, R64, R69, R74, R79, R9: value 10k -> 4.7k
Connections:
- net /MCXN947_MCU/P0-3/P5_5 renamed /SHIFT_REG_LAT
- net /MCXN947_MCU/P5-4 renamed /SHIFT_REG_OE
- J1 pad 15: /I2C_SCL1 -> /MCXN947_MCU/P3-21/SAI1_RXD0
- J1 pad 5: /I2C_SDA1 -> /MCXN947_MCU/P3-20/SAI1_TXD0
- J1 pad 6: /DISPLAY_CS -> /MCXN947_MCU/P1-23/P2-6
- J2 pad 10: /MOS_12_ON -> /MCXN947_MCU/P0-26/FC1-SDI
- J2 pad 12: /MOS_11_ON -> /DISPLAY_SCK
- J2 pad 18: /MOS_10_ON -> /I2C_SDA1
- J2 pad 2: /MOS_16_ON -> /DISPLAY_DC
- J2 pad 20: /MOS_9_ON -> /I2C_SCL1
- J2 pad 3: /MOS_8_ON -> /MCXN947_MCU/P5-2/P0-14
- J2 pad 4: /MOS_15_ON -> /DISPLAY_RST
- J2 pad 6: /MOS_14_ON -> /DISPLAY_CS
- J2 pad 8: /MOS_13_ON -> /DISPLAY_MOSI
- J4 pad 1: /MOS_5_ON -> /MCXN947_MCU/P4-12/P0-21
- J4 pad 10: /MOS_3_ON -> /SHIFT_REG_CLR
- J4 pad 12: /MOS_4_ON -> /MCXN947_MCU/P0-23/P1-22
- J4 pad 3: /MOS_6_ON -> /MCXN947_MCU/OP-0-I/P0-20
- J4 pad 5: /MOS_7_ON -> /MCXN947_MCU/P4-16/P0-18
- J4 pad 6: /MOS_1_ON -> /SHIFT_REG_SER
- J4 pad 8: /MOS_2_ON -> /SHIFT_REG_CLK
- J9 pad 13: /DISPLAY_DC -> /MCXN947_MCU/P1_11/EZH_LCD_D7_CAMERA_D7
- J9 pad 15: /DISPLAY_SCK -> /MCXN947_MCU/P0_5/EZH_CAMERA_PCLK
- J9 pad 17: /DISPLAY_MOSI -> /MCXN947_MCU/P0_4/EZH_CAMERA_VSYNC
- J9 pad 5: /DISPLAY_RST -> /MCXN947_MCU/P1_19/EZH_LCD_D15_CAMERA_RST

Commit message: -add some more pinning changes, add rts flow control for rs485
Parts:
- removed H1: M4 Shielding Hole, MountingHole:MOUNTINGHOLE_3.2MM_M3
- added H2: MountingHole, MountingHole:MountingHole_3.2mm_M3, F.Cu at (238.9, 65.8)
- added H3: MountingHole, MountingHole:MountingHole_3.2mm_M3, F.Cu at (262.5, 84.1)
- added H4: MountingHole, MountingHole:MountingHole_3.2mm_M3, F.Cu at (262.5, 92.0)
- added H5: MountingHole, MountingHole:MountingHole_3.2mm_M3, F.Cu at (262.5, 100.0)
- added U36: 74HC595, Package_SO:SOIC-16_3.9x9.9mm_P1.27mm, F.Cu at (24.6, 113.1)
- added U37: 74HC595, Package_SO:SOIC-16_3.9x9.9mm_P1.27mm, F.Cu at (33.0, 113.1)
- J7: value +24V -> Barrel_Jack_MountingPin
- moved D13 42.3 mm to (65.8, 101.4)
- moved D16 42.3 mm to (66.6, 60.5)
- moved Q13 42.3 mm to (70.0, 96.8)
- moved R60 42.3 mm to (70.6, 110.6)
- moved R61 42.3 mm to (70.6, 108.1)
- moved R62 42.3 mm to (70.6, 105.5)
- moved R63 42.3 mm to (70.6, 103.0)
- moved R64 42.3 mm to (70.6, 100.5)
- moved R77 42.3 mm to (70.1, 77.1)
- moved R78 42.3 mm to (70.1, 74.6)
- moved R79 42.3 mm to (70.1, 72.0)
- moved R11 42.3 mm to (66.8, 84.0)
- moved R13 42.3 mm to (72.1, 88.0)
- moved R75 42.3 mm to (66.2, 76.6)
- moved D3 42.3 mm to (67.2, 90.3)
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Connections:
- IC3 pad 7: /I2C_SCL -> +3V3
- IC4 pad 5: GND -> +3V3
- IC4 pad 6: +3V3 -> GND
- IC4 pad 7: /I2C_SDA -> GND
- IC6 pad 7: /I2C_SCL -> +3V3
- IC7 pad 7: /I2C_SDA -> GND
- J1 pad 2: /RS485_RXD -> /MCXN947_MCU/P4-3/RXD2
- J1 pad 4: /RS485_TXD -> /MCXN947_MCU/P4-2/TXD2
- J2 pad 15: /MCXN947_MCU/P1-1/TSI0_CH1 -> /I2C_SCL1
- J2 pad 17: /MCXN947_MCU/P1-0/TSI0_CH0 -> /I2C_SDA1
- J2 pad 18: /I2C_SDA1 -> /MCXN947_MCU/P4-0/P1-16
- J2 pad 20: /I2C_SCL1 -> /MCXN947_MCU/P4-1/P1-17
- J7 pad 3: (no net) -> GND
- J9 pad 3: /MCXN947_MCU/P1_17/EZH_LCD_D13 -> /RS485_TXD
- J9 pad 4: /MCXN947_MCU/P1_16/EZH_LCD_D12 -> /RS485_RXD
- J9 pad 6: /MCXN947_MCU/P1_18/EZH_LCD_D14_CAMERA_PDOWN -> /RS485_RTS
- U33 pad 2: /RS485_RE -> /RS485_RTS
- U33 pad 3: /RS485_DE -> /RS485_RTS

Commit message: -enh final revision; ordered
Parts:
- removed F4: Fuse, Fuse:Fuse_2920_7451Metric_Pad2.10x5.45mm_HandSolder
- removed the H2 at (134.2, 64.4)
- removed the H3 at (134.2, 113.4)
- removed the H4 at (237.7, 112.8)
- removed R113: 4.7k, Resistor_SMD:R_0603_1608Metric_Pad0.98x0.95mm_HandSolder
- added C10: 100n, Capacitor_SMD:C_0603_1608Metric_Pad1.08x0.95mm_HandSolder, F.Cu at (167.1, 85.1)
- added C11: 100n, Capacitor_SMD:C_0603_1608Metric_Pad1.08x0.95mm_HandSolder, F.Cu at (189.9, 85.3)
- added C12: 100n, Capacitor_SMD:C_0603_1608Metric_Pad1.08x0.95mm_HandSolder, F.Cu at (211.2, 93.2)
- added C13: 100n, Capacitor_SMD:C_0603_1608Metric_Pad1.08x0.95mm_HandSolder, F.Cu at (189.8, 91.3)
- added C14: 100n, Capacitor_SMD:C_0603_1608Metric_Pad1.08x0.95mm_HandSolder, F.Cu at (234.5, 65.6)
- added C15: 100n, Capacitor_SMD:C_0603_1608Metric_Pad1.08x0.95mm_HandSolder, F.Cu at (152.0, 109.2)
- added C16: 100n, Capacitor_SMD:C_0603_1608Metric_Pad1.08x0.95mm_HandSolder, B.Cu at (237.1, 65.5)
- added C17: 100n, Capacitor_SMD:C_0603_1608Metric_Pad1.08x0.95mm_HandSolder, F.Cu at (240.3, 128.8)
- added C9: 100n, Capacitor_SMD:C_0603_1608Metric_Pad1.08x0.95mm_HandSolder, F.Cu at (192.4, 111.3)
- added H1: M4 Shielding Hole, MountingHole:MountingHole_3.2mm_M3_ISO14580_Pad_TopBottom, F.Cu at (258.3, 132.1)
- added IC10: P3T1755DPZ, Library:P3T1755DPZ, B.Cu at (111.2, 86.4)
- added REF**: MountingHole_3.2mm_M3, MountingHole:MountingHole_3.2mm_M3, F.Cu at (111.4, 135.2)
- added REF**: MountingHole_3.2mm_M3, MountingHole:MountingHole_3.2mm_M3, F.Cu at (111.4, 54.1)
- D1, D11, D13, D15, D3, D5, D7, D9, H2, H3, H4, H5, IC3, IC8, IC9, Q11, Q13, Q15, Q2, Q3, Q5, Q7, Q9, R10, R107, R108, R109, R11, R110, R12, R13, R14, R20, R21, R22, R23, R24, R30, R31, R32, R33, R34, R40, R41, R42, R43, R44, R50, R51, R52, R53, R54, R60, R61, R62, R63, R64, R70, R71, R72, R73, R74, R80: moved to B.Cu
- J1, J12, J2, J3, J4, J9: moved to F.Cu
- U10, U13, U14, U17, U18, U21, U22, U25, U26, U29, U3, U30, U4, U5, U6, U9: footprint Package_DIP:DIP-4_W7.62mm -> Package_DIP:DIP-4_W7.62mm_SMDSocket_SmallPads; moved to B.Cu
- U11, U12, U15, U16, U19, U20, U23, U24, U27, U28, U31, U32, U34, U35, U7, U8: footprint Package_DIP:DIP-4_W7.62mm -> Package_DIP:DIP-4_W7.62mm_SMDSocket_SmallPads
- moved IC9 240.4 mm to (250.6, 123.8)
- moved IC5 233.4 mm to (242.3, 120.1), turned to 180 degrees
- moved R106 232.1 mm to (241.3, 87.6), turned to -90 degrees
- moved R103 228.5 mm to (237.7, 79.7)
- moved IC8 227.0 mm to (236.7, 120.5)
- moved R104 226.5 mm to (235.9, 78.2)
- moved D17 225.4 mm to (173.4, 37.9)
- moved R105 224.2 mm to (233.7, 76.7)
- moved R99 224.1 mm to (186.5, 38.4), turned to 180 degrees
- moved Q17 222.9 mm to (194.9, 38.9), turned to 180 degrees
- moved R96 221.9 mm to (203.8, 37.9), turned to 180 degrees
- moved J5 219.6 mm to (236.0, 124.0)
- moved R97 216.1 mm to (197.4, 35.7)
- moved R93 214.0 mm to (188.6, 109.0), turned to 180 degrees
- moved C1 212.3 mm to (190.7, 43.5), turned to -90 degrees
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Connections:
- F2 pad 1: Net-(F2-Pad1) -> Net-(IC2-VDD)
- IC5 pad 1: /DISPLAY_RST -> /DISPLAY_MOSI
- IC5 pad 5: /DISPLAY_MOSI -> /DISPLAY_RST
- J12 pad 17: /MCU_MOS_6_IN -> /MOS_10_ON
- J12 pad 18: /MCU_MOS_7_IN -> /MOS_16_ON
- J12 pad 19: /MCU_MOS_8_IN -> /MOS_8_ON
- J12 pad 20: /MOS_9_IN -> /MOS_9_ON
- J12 pad 21: /MCU_MOS_10_IN -> /MOS_6_ON
- J12 pad 22: /MOS_11_IN -> /MOS_7_ON
- J12 pad 23: /MCU_MOS_12_IN -> /MOS_4_ON
- J12 pad 24: /MOS_13_IN -> /MOS_5_ON
- J12 pad 25: /MCU_MOS_14_IN -> /MOS_2_ON
- J12 pad 26: /MOS_15_IN -> /MOS_3_ON
- J12 pad 27: /MCU_MOS_16_IN -> /MOS_1_ON
- J12 pad 3: /MCU_MOS_2_IN -> /MOS_11_ON
- J12 pad 4: /MCU_MOS_1_IN -> /MOS_15_ON
- J12 pad 5: /MCU_MOS_4_IN -> /MOS_14_ON
- J12 pad 6: /MCU_MOS_3_IN -> /MOS_13_ON
- J12 pad 7: /MCU_MOS_5_IN -> /MOS_12_ON
- R1 pad 1: /MCU_MOS_2_IN -> /MOS_2_IN
- R15 pad 1: /MCU_MOS_4_IN -> /MOS_4_IN
- R25 pad 1: /MCU_MOS_6_IN -> /MOS_6_IN
- R35 pad 1: /MCU_MOS_8_IN -> /MOS_8_IN
- R45 pad 1: /MCU_MOS_10_IN -> /MOS_10_IN
- R55 pad 1: /MCU_MOS_12_IN -> /MOS_12_IN
- R65 pad 1: /MCU_MOS_14_IN -> /MOS_14_IN
- R75 pad 1: /MCU_MOS_16_IN -> /MOS_16_IN
- U1 pad 10: Net-(R81-Pad1) -> Net-(R83-Pad1)
- U1 pad 11: /MOS_7_IN -> /MOS_5_IN
- U1 pad 12: /MCU_MOS_7_IN -> /MCU_MOS_5_IN
- U1 pad 13: Net-(R83-Pad1) -> Net-(R81-Pad1)
- U1 pad 8: /MOS_5_IN -> /MOS_7_IN
- U1 pad 9: /MCU_MOS_5_IN -> /MCU_MOS_7_IN
- U2 pad 10: Net-(R87-Pad1) -> Net-(R85-Pad1)
- U2 pad 11: /MOS_15_IN -> /MOS_13_IN
- U2 pad 12: /MCU_MOS_15_IN -> /MCU_MOS_13_IN
- U2 pad 13: Net-(R85-Pad1) -> Net-(R87-Pad1)
- U2 pad 8: /MOS_13_IN -> /MOS_15_IN
- U2 pad 9: /MCU_MOS_13_IN -> /MCU_MOS_15_IN
- U36 pad 1: /MOS_2_ON -> /MOS_2_IN
- U36 pad 15: /MOS_1_ON -> /MCU_MOS_1_IN
- U36 pad 2: /MOS_3_ON -> /MCU_MOS_3_IN
- U36 pad 3: /MOS_4_ON -> /MOS_4_IN
- U36 pad 4: /MOS_5_ON -> /MCU_MOS_5_IN
- U36 pad 5: /MOS_6_ON -> /MOS_6_IN
- U36 pad 6: /MOS_7_ON -> /MCU_MOS_7_IN
- U36 pad 7: /MOS_8_ON -> /MOS_8_IN
- U37 pad 1: /MOS_10_ON -> /MOS_10_IN
- U37 pad 15: /MOS_9_ON -> /MCU_MOS_9_IN
- U37 pad 2: /MOS_11_ON -> /MCU_MOS_11_IN
- U37 pad 3: /MOS_12_ON -> /MOS_12_IN
- U37 pad 4: /MOS_13_ON -> /MCU_MOS_13_IN
- U37 pad 5: /MOS_14_ON -> /MOS_14_IN
- U37 pad 6: /MOS_15_ON -> /MCU_MOS_15_IN
- U37 pad 7: /MOS_16_ON -> /MOS_16_IN
Routing:
- net +3V3: track 0.00 -> 878.1 mm, vias 0 -> 33
- net GND: track 0.00 -> 354.7 mm, vias 0 -> 328
- net +24V: track 0.00 -> 284.7 mm, vias 0 -> 48
- net /I2C_SDA: track 0.00 -> 233.3 mm, vias 0 -> 3
- net +5V: track 0.00 -> 227.2 mm, vias 0 -> 3
- net /I2C_SCL: track 0.00 -> 224.6 mm, vias 0 -> 3
- net /TEMP_ALERT: track 0.00 -> 169.3 mm, vias 0 -> 5
- net /VOLT_MEAS_BATT: track 0.00 -> 128.8 mm, vias 0 -> 1
- net /RS485_B: track 0.00 -> 128.3 mm
- net /MOS_2_ON: track 0.00 -> 118.9 mm, vias 0 -> 3
- net /RS485_A: track 0.00 -> 118.2 mm
- net /MOS_1_IN: track 0.00 -> 102.6 mm, vias 0 -> 1
- net /MOS_11_IN: track 0.00 -> 102.5 mm, vias 0 -> 1
- net /MOS_16_IN: track 0.00 -> 95.8 mm
- net /MOS_16_ON: track 0.00 -> 93.6 mm, vias 0 -> 1
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- added copper zone on B.Cu, net GND
- added copper zone on F.Cu, net GND
- added copper zone on In1.Cu, net GND
- added copper zone on In2.Cu, net GND
Other:
- board size 160 x 103 mm -> 220.1 x 120.3 mm
- copper layers 2 -> 4
- board text added: "- +"
- board text added: "3.3"
- board text added: "A"
- board text added: "B"
- board text added: "B LED"
- board text added: "BATTERY"
- board text added: "BL"
- board text added: "CS"
- board text added: "DC"
- board text added: "DISP_KEYPAD"
- board text added: "Fuse 2A F"
- board text added: "G LED"
- board text added: "GND"
- board text added: "I2C SCL"
- board text added: "I2C SDA"
- board text added: "KEY INT"
- board text added: "KEY RST"
- board text added: "P LED"
- board text added: "R LED"
- board text added: "RS485"
- board text added: "RST"
- board text added: "SPI DO"
- board text added: "SPI SCK"
- board text added: "Status and PWR LED"
- board text added: "VCC"
- board text removed: "Note: The positioning of the connectors in the PCB are at coordinates that seem {dblquote}off{dblquote} by 2-6mil. This was a design bug in the FRDM-MCX947 PCB design. The connectors don't quite match to true arduino positioning, but are close enough that boards will mate."
