File: hardware/GridSwitcher_PCB/mcxn947.kicad_sch (KiCad schematic)
At the start: 6 parts, among them J1 ${ALTIUM_VALUE}, J2 ${ALTIUM_VALUE}, J3 ${ALTIUM_VALUE}, J4 ${ALTIUM_VALUE}, J5 ${ALTIUM_VALUE}, J6 ${ALTIUM_VALUE}

Commit message: -enh made some progress on pcb/fp design
Parts:
- J1: renamed from J5; footprint (none) -> Connector_PinHeader_2.54mm:PinHeader_2x08_P2.54mm_Vertical
- J12: renamed from J1; footprint (none) -> Connector_PinHeader_2.54mm:PinHeader_2x14_P2.54mm_Vertical
- J2: renamed from J4; footprint (none) -> Connector_PinHeader_2.54mm:PinHeader_2x10_P2.54mm_Vertical
- J3: renamed from J2; footprint (none) -> Connector_PinHeader_2.54mm:PinHeader_2x08_P2.54mm_Vertical
- J4: renamed from J3; footprint (none) -> Connector_PinHeader_2.54mm:PinHeader_2x06_P2.54mm_Vertical
- J9: renamed from J6; footprint (none) -> Connector_PinHeader_2.54mm:PinHeader_2x16_P2.54mm_Vertical
Changed lines of the file:
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@@
   (symbol (lib_id "FRDM-MCXN947__Shield_Template-altium-import:root_2_mirrored_SSQ-110-03-T-D") (at 209.55 46.99 0) (unit 1)
     (in_bom yes) (on_board yes) (dnp no)
-    (property "Reference" "J4" (at 205.74 33.02 0)
+    (property "Reference" "J2" (at 205.74 33.02 0)
       (effects (font (size 1.27 1.27)) (justify left bottom))
     )
@@
       (effects (font (size 1.27 1.27)) (justify left bottom))
     )
-    (property "Footprint" "" (at 209.55 46.99 0)
+    (property "Footprint" "Connector_PinHeader_2.54mm:PinHeader_2x10_P2.54mm_Vertical" (at 209.55 46.99 0)
       (effects (font (size 1.27 1.27)) hide)
     )
@@
       (project "GridSwitcher_PCB"
         (path "/85d790fa-2a68-4a26-9dd2-3e7bd6cf9669/fc33dd87-afec-4399-b566-7d146648c6e3"
-          (reference "J4") (unit 1)
+          (reference "J2") (unit 1)
         )
       )
@@
   (symbol (lib_id "FRDM-MCXN947__Shield_Template-altium-import:root_2_mirrored_SSQ-108-03-T-D") (at 209.55 82.55 0) (unit 1)
     (in_bom yes) (on_board yes) (dnp no)
-    (property "Reference" "J5" (at 205.74 71.12 0)
+    (property "Reference" "J1" (at 205.74 71.12 0)
       (effects (font (size 1.27 1.27)) (justify left bottom))
     )
@@
       (effects (font (size 1.27 1.27)) (justify left bottom))
     )
-    (property "Footprint" "" (at 209.55 82.55 0)
+    (property "Footprint" "Connector_PinHeader_2.54mm:PinHeader_2x08_P2.54mm_Vertical" (at 209.55 82.55 0)
       (effects (font (size 1.27 1.27)) hide)
     )
@@
       (project "GridSwitcher_PCB"
         (path "/85d790fa-2a68-4a26-9dd2-3e7bd6cf9669/fc33dd87-afec-4399-b566-7d146648c6e3"
-          (reference "J5") (unit 1)
+          (reference "J1") (unit 1)
         )
       )
@@
   (symbol (lib_id "FRDM-MCXN947__Shield_Template-altium-import:root_0_mirrored_SSQ-116-03-T-D") (at 212.09 135.89 0) (unit 1)
     (in_bom yes) (on_board yes) (dnp no)
-    (property "Reference" "J6" (at 208.28 116.84 0)
+    (property "Reference" "J9" (at 208.28 116.84 0)
       (effects (font (size 1.27 1.27)) (justify left bottom))
     )
@@
       (effects (font (size 1.27 1.27)) (justify left bottom))
     )
-    (property "Footprint" "" (at 212.09 135.89 0)
+    (property "Footprint" "Connector_PinHeader_2.54mm:PinHeader_2x16_P2.54mm_Vertical" (at 212.09 135.89 0)
       (effects (font (size 1.27 1.27)) hide)
     )
@@
       (project "GridSwitcher_PCB"
         (path "/85d790fa-2a68-4a26-9dd2-3e7bd6cf9669/fc33dd87-afec-4399-b566-7d146648c6e3"
-          (reference "J6") (unit 1)
+          (reference "J9") (unit 1)
         )
       )
@@
   (symbol (lib_id "FRDM-MCXN947__Shield_Template-altium-import:root_0_mirrored_SSQ-114-03-T-D") (at 60.96 144.78 0) (unit 1)
     (in_bom yes) (on_board yes) (dnp no)
-    (property "Reference" "J1" (at 57.15 129.54 0)
+    (property "Reference" "J12" (at 57.15 129.54 0)
       (effects (font (size 1.27 1.27)) (justify left bottom))
     )
@@
       (effects (font (size 1.27 1.27)) (justify left bottom))
     )
-    (property "Footprint" "" (at 60.96 144.78 0)
+    (property "Footprint" "Connector_PinHeader_2.54mm:PinHeader_2x14_P2.54mm_Vertical" (at 60.96 144.78 0)
       (effects (font (size 1.27 1.27)) hide)
     )
@@
       (project "GridSwitcher_PCB"
         (path "/85d790fa-2a68-4a26-9dd2-3e7bd6cf9669/fc33dd87-afec-4399-b566-7d146648c6e3"
-          (reference "J1") (unit 1)
+          (reference "J12") (unit 1)
         )
       )
@@
   (symbol (lib_id "FRDM-MCXN947__Shield_Template-altium-import:root_0_mirrored_SSQ-108-03-T-D") (at 71.12 36.83 0) (unit 1)
     (in_bom yes) (on_board yes) (dnp no)
-    (property "Reference" "J2" (at 67.31 27.94 0)
+    (property "Reference" "J3" (at 67.31 27.94 0)
       (effects (font (size 1.27 1.27)) (justify left bottom))
     )
@@
       (effects (font (size 1.27 1.27)) (justify left bottom))
     )
-    (property "Footprint" "" (at 71.12 36.83 0)
+    (property "Footprint" "Connector_PinHeader_2.54mm:PinHeader_2x08_P2.54mm_Vertical" (at 71.12 36.83 0)
       (effects (font (size 1.27 1.27)) hide)
     )
@@
       (project "GridSwitcher_PCB"
         (path "/85d790fa-2a68-4a26-9dd2-3e7bd6cf9669/fc33dd87-afec-4399-b566-7d146648c6e3"
-          (reference "J2") (unit 1)
+          (reference "J3") (unit 1)
         )
       )
@@
   (symbol (lib_id "FRDM-MCXN947__Shield_Template-altium-import:root_0_mirrored_SSQ-106-03-T-D") (at 71.12 78.74 0) (unit 1)
     (in_bom yes) (on_board yes) (dnp no)
-    (property "Reference" "J3" (at 67.31 72.39 0)
+    (property "Reference" "J4" (at 67.31 72.39 0)
       (effects (font (size 1.27 1.27)) (justify left bottom))
     )
@@
       (effects (font (size 1.27 1.27)) (justify left bottom))
     )
-    (property "Footprint" "" (at 71.12 78.74 0)
+    (property "Footprint" "Connector_PinHeader_2.54mm:PinHeader_2x06_P2.54mm_Vertical" (at 71.12 78.74 0)
       (effects (font (size 1.27 1.27)) hide)
     )
@@
       (project "GridSwitcher_PCB"
         (path "/85d790fa-2a68-4a26-9dd2-3e7bd6cf9669/fc33dd87-afec-4399-b566-7d146648c6e3"
-          (reference "J3") (unit 1)
-        )
-      )
+          (reference "J4") (unit 1)
+        )
+      )

Commit message: -enh final revision; ordered
Parts:
- added C15, C16, C17: 100n, Capacitor_SMD:C_0603_1608Metric_Pad1.08x0.95mm_HandSolder, symbol Device:C_Small
Connections:
- net +3V3: now also C15.2, C16.2, C17.2
- net GND: now also C15.1, C16.1, C17.1
