File: hardware/GridSwitcher_PCB/mosfet_drivers.kicad_sch (KiCad schematic)
At the start: 3 parts, among them IC3 P3T1755DPZ, IC4 P3T1755DPZ, IC7 P3T1755DPZ

Commit message: -enh made some progress on pcb/fp design
Parts:
- IC3, IC4, IC7: footprint (none) -> Library:P3T1755DPZ
Changed lines of the file:
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@@
       (effects (font (size 1.27 1.27)))
     )
-    (property "Footprint" "" (at 266.7 149.53 0)
+    (property "Footprint" "Library:P3T1755DPZ" (at 266.7 149.53 0)
       (effects (font (size 1.27 1.27)) (justify left top) hide)
     )
@@
       (effects (font (size 1.27 1.27)))
     )
-    (property "Footprint" "" (at 266.7 120.32 0)
+    (property "Footprint" "Library:P3T1755DPZ" (at 266.7 120.32 0)
       (effects (font (size 1.27 1.27)) (justify left top) hide)
     )
@@
       (effects (font (size 1.27 1.27)))
     )
-    (property "Footprint" "" (at 266.7 180.01 0)
+    (property "Footprint" "Library:P3T1755DPZ" (at 266.7 180.01 0)
       (effects (font (size 1.27 1.27)) (justify left top) hide)
     )

Commit message: -add some more pinning changes, add rts flow control for rs485
Connections:
- net +3V3: now also IC3.7 (A0), IC4.5 (A2); no longer IC4.6 (A1)
- net GND: now also IC4.6 (A1), IC4.7 (A0), IC7.7 (A0); no longer IC4.5 (A2)
- net I2C_SCL: no longer IC3.7 (A0)
- net I2C_SDA: no longer IC4.7 (A0), IC7.7 (A0)
Changed lines of the file:
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@@
+	)
+	(junction
+		(at 270.51 38.1)
+		(diameter 0)
+		(color 0 0 0 0)
 	)
 	(junction
@@
 	)
 	(junction
+		(at 275.59 90.17)
+		(diameter 0)
+		(color 0 0 0 0)
+	)
+	(junction
 		(at 240.03 67.31)
 		(diameter 0)
 		(color 0 0 0 0)
 	)
+	(junction
+		(at 273.05 57.15)
+		(diameter 0)
+		(color 0 0 0 0)
+	)
 	(wire
 		(pts
@@
 	(wire
 		(pts
+			(xy 273.05 57.15) (xy 273.05 54.61)
+		)
+		(stroke
+			(width 0)
+			(type default)
+		)
+	)
+	(wire
+		(pts
 			(xy 68.58 106.68) (xy 68.58 107.95)
 		)
@@
 	(wire
 		(pts
+			(xy 271.78 27.94) (xy 271.78 38.1)
+		)
+		(stroke
+			(width 0)
+			(type default)
+		)
+	)
+	(wire
+		(pts
 			(xy 129.54 30.48) (xy 127 30.48)
 		)
@@
 	(wire
 		(pts
-			(xy 271.78 85.09) (xy 270.51 85.09)
+			(xy 270.51 85.09) (xy 273.05 85.09)
+		)
+		(stroke
+			(width 0)
+			(type default)
+		)
+	)
+	(wire
+		(pts
+			(xy 275.59 87.63) (xy 275.59 90.17)
 		)
 		(stroke
@@
 	(wire
 		(pts
-			(xy 270.51 90.17) (xy 271.78 90.17)
-		)
-		(stroke
-			(width 0)
-			(type default)
-		)
-	)
-	(wire
-		(pts
 			(xy 270.51 59.69) (xy 273.05 59.69)
 		)
@@
 	(wire
 		(pts
-			(xy 273.05 59.69) (xy 273.05 54.61)
+			(xy 273.05 59.69) (xy 273.05 57.15)
 		)
 		(stroke
@@
 	(wire
 		(pts
+			(xy 270.51 92.71) (xy 273.05 92.71)
+		)
+		(stroke
+			(width 0)
+			(type default)
+		)
+	)
+	(wire
+		(pts
 			(xy 127 156.21) (xy 129.54 156.21)
 		)
@@
 	(wire
 		(pts
-			(xy 275.59 57.15) (xy 270.51 57.15)
+			(xy 273.05 57.15) (xy 270.51 57.15)
 		)
 		(stroke
@@
 	(wire
 		(pts
-			(xy 274.32 27.94) (xy 270.51 27.94)
+			(xy 271.78 27.94) (xy 270.51 27.94)
 		)
 		(stroke
@@
 	(wire
 		(pts
+			(xy 270.51 87.63) (xy 275.59 87.63)
+		)
+		(stroke
+			(width 0)
+			(type default)
+		)
+	)
+	(wire
+		(pts
 			(xy 240.03 97.79) (xy 240.03 92.71)
 		)
@@
 	(wire
 		(pts
+			(xy 270.51 90.17) (xy 275.59 90.17)
+		)
+		(stroke
+			(width 0)
+			(type default)
+		)
+	)
+	(wire
+		(pts
 			(xy 129.54 29.21) (xy 129.54 30.48)
 		)
@@
 	(wire
 		(pts
-			(xy 270.51 92.71) (xy 270.51 97.79)
-		)
-		(stroke
-			(width 0)
-			(type default)
-		)
-	)
-	(wire
-		(pts
 			(xy 95.25 77.47) (xy 100.33 77.47)
 		)
@@
 	(wire
 		(pts
+			(xy 273.05 92.71) (xy 273.05 85.09)
+		)
+		(stroke
+			(width 0)
+			(type default)
+		)
+	)
+	(wire
+		(pts
 			(xy 273.05 54.61) (xy 270.51 54.61)
 		)
@@
 	(wire
 		(pts
+			(xy 271.78 38.1) (xy 270.51 38.1)
+		)
+		(stroke
+			(width 0)
+			(type default)
+		)
+	)
+	(wire
+		(pts
 			(xy 240.03 69.85) (xy 240.03 67.31)
 		)
@@
 	(wire
 		(pts
-			(xy 273.05 87.63) (xy 270.51 87.63)
-		)
-		(stroke
-			(width 0)
-			(type default)
-		)
-	)
-	(wire
-		(pts
 			(xy 68.58 35.56) (xy 68.58 36.83)
 		)
@@
 	(wire
 		(pts
+			(xy 275.59 90.17) (xy 275.59 97.79)
+		)
+		(stroke
+			(width 0)
+			(type default)
+		)
+	)
+	(wire
+		(pts
 			(xy 270.51 33.02) (xy 270.51 38.1)
 		)
@@
 	(wire
 		(pts
-			(xy 271.78 90.17) (xy 271.78 85.09)
-		)
-		(stroke
-			(width 0)
-			(type default)
-		)
-	)
-	(wire
-		(pts
 			(xy 129.54 52.07) (xy 129.54 53.34)
 		)
@@
 	(wire
 		(pts
-			(xy 240.03 97.79) (xy 270.51 97.79)
+			(xy 240.03 97.79) (xy 275.59 97.79)
 		)
 		(stroke
@@
 		)
 	)
-	(hierarchical_label "I2C_SCL"
-		(shape input)
-		(at 275.59 57.15 0)
-		(fields_autoplaced yes)
-		(effects
-			(font
-				(size 1.27 1.27)
-			)
-			(justify left)
-		)
-	)
 	(hierarchical_label "MOS_3_ON"
 		(shape output)
@@
 		)
 	)
-	(hierarchical_label "I2C_SDA"
-		(shape input)
-		(at 273.05 87.63 0)
-		(fields_autoplaced yes)
-		(effects
-			(font
-				(size 1.27 1.27)
-			)
-			(justify left)
-		)
-	)
 	(hierarchical_label "MOS_2_ON"
 		(shape output)
@@
 		)
 	)
-	(hierarchical_label "I2C_SDA"
-		(shape input)
-		(at 274.32 27.94 0)
-		(fields_autoplaced yes)
-		(effects
-			(font
-				(size 1.27 1.27)
-			)
-			(justify left)
-		)
-	)

Commit message: -enh final revision; ordered
Parts:
- added IC10: P3T1755DPZ, Library:P3T1755DPZ, symbol P3T1755DPZ:P3T1755DPZ
Connections:
- net +3V3: now also IC10.5 (A2), IC10.7 (A0), IC10.8 (VCC)
- net GND: now also IC10.4 (GND), IC10.6 (A1)
- net I2C_SCL: now also IC10.2 (SCL)
- net I2C_SDA: now also IC10.1 (SDA)
- net TEMP_ALERT: now also IC10.3 (~{ALERT})
Other:
- note added: "I2C Adr: IC7: 0b1000 010 IC3: 0b1000 011 IC4: 0b1000 100 IC10: 0b1000 101"
